Commit message: Fix the urdf of franka hand with new long fingers

File: franka_description/urdf/panda_arm_hand_with_long_fingers.urdf (robot description, URDF)
Before this commit: robot panda, 12 links, 11 joints
Links:
- link panda_leftfinger: geometry collision mesh filename=package://drake_models/franka_description/meshes/visual/lon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; visual mesh filename=package://drake_models/franka_description/meshes/visual/fin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
- link panda_rightfinger: geometry collision mesh filename=package://drake_models/franka_description/meshes/visual/lon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; visual mesh filename=package://drake_models/franka_description/meshes/visual/fin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

Commit message: Add fake link at the fingertips of franka hand for frame visualization purpose

File: franka_description/urdf/panda_arm_hand_with_long_fingers.urdf (robot description, URDF)
Before this commit: robot panda, 12 links, 11 joints
Links:
- added link finger_tip
Joints:
- added joint finger_tip_joint: type fixed, parent panda_hand, child finger_tip, origin xyz=0 0 0.203191 rpy=0 0 0
