Commit message: Fix the pose of the finger tip frame

File: franka_description/urdf/panda_arm_hand_with_fixed_long_fingers.urdf (robot description, URDF)
Before this commit: robot panda, 13 links, 12 joints
Joints:
- joint finger_tip_joint: origin xyz=0 0 0.203191 rpy=0 0 0 -> xyz=0 0 0.203191 rpy=3.14159 0 0

File: franka_description/urdf/panda_arm_hand_with_long_fingers.urdf (robot description, URDF)
Before this commit: robot panda, 13 links, 12 joints
Joints:
- joint finger_tip_joint: origin xyz=0 0 0.203191 rpy=0 0 0 -> xyz=0 0 0.203191 rpy=3.14159 0 0

Commit message: fix: shift upward slightly the finger_tip frame of panda hand models

File: franka_description/urdf/panda_arm_hand_with_fixed_long_fingers.urdf (robot description, URDF)
Before this commit: robot panda, 13 links, 12 joints
Joints:
- joint finger_tip_joint: origin xyz=0 0 0.203191 rpy=3.14159 0 0 -> xyz=0 0 0.198191 rpy=3.14159 0 0

File: franka_description/urdf/panda_arm_hand_with_long_fingers.urdf (robot description, URDF)
Before this commit: robot panda, 13 links, 12 joints
Joints:
- joint finger_tip_joint: origin xyz=0 0 0.203191 rpy=3.14159 0 0 -> xyz=0 0 0.198191 rpy=3.14159 0 0

File: franka_description/urdf/panda_hand_with_fixed_long_fingers.urdf (robot description, URDF)
Before this commit: robot panda_hand_with_long_fingers, 5 links, 4 joints
Joints:
- joint finger_tip_joint: origin xyz=0 0 0.203191 rpy=3.14159 0 0 -> xyz=0 0 0.198191 rpy=3.14159 0 0

File: franka_description/urdf/panda_hand_with_long_fingers.urdf (robot description, URDF)
Before this commit: robot panda_hand_with_long_fingers, 5 links, 4 joints
Joints:
- joint finger_tip_joint: origin xyz=0 0 0.203191 rpy=3.14159 0 0 -> xyz=0 0 0.198191 rpy=3.14159 0 0
