Commit message: fix the rerun urdf to the non-fixed finger panda

File: franka_description/urdf/panda_arm_hand_with_long_fingers_paths_resolved.urdf (robot description, URDF)
Before this commit: robot panda, 13 links, 12 joints
Links:
- link panda_hand: geometry collision sphere radius=0.05; collision sphere radius=0.05
- link panda_leftfinger: geometry collision mesh filename=models/franka_description/meshes/visual/long_finger.obj; visual mesh filename=models/franka_description/meshes/visual/finger_holder.obj
- link panda_link0: geometry collision sphere radius=0.06; collision sphere radius=0.06
- link panda_link1: geometry collision sphere radius=0.06; collision sphere radius=0.06
- link panda_link2: geometry collision sphere radius=0.06; collision sphere radius=0.06
- link panda_link3: geometry collision sphere radius=0.06; collision sphere radius=0.06
- link panda_link4: geometry collision sphere radius=0.05; collision sphere radius=0.055
- link panda_link5: geometry collision sphere radius=0.035; collision sphere radius=0.035
- link panda_link6: geometry collision sphere radius=0.05; collision sphere radius=0.06
- link panda_link7: geometry collision sphere radius=0.05; collision sphere radius=0.06
- link panda_link8: geometry collision sphere radius=0.04
- link panda_rightfinger: geometry collision mesh filename=models/franka_description/meshes/visual/long_finger.obj; visual mesh filename=models/franka_description/meshes/visual/finger_holder.obj
Joints:
- joint panda_finger_joint1: type fixed -> prismatic
- joint panda_finger_joint2: type fixed -> prismatic

Commit message: match changes in rerun urdf

File: franka_description/urdf/panda_arm_hand_with_long_fingers_paths_resolved.urdf (robot description, URDF)
Before this commit: robot panda, 13 links, 12 joints
Joints:
- joint finger_tip_joint: origin xyz=0 0 0.203191 rpy=3.14159 0 0 -> xyz=0 0 0.198191 rpy=3.14159 0 0
